File: LGM-01/licznik.brd (EAGLE design)
At the start: 100 x 80 mm, 60 parts, among them IC1 7805L, IC2 NE555, Q1 BC177, Q10 BC107, Q11 BC107, Q12 BC177, Q13 BC107, Q14 BC107, Q15 IRF840, Q16 BC177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

Commit message: edycje
Parts:
- moved R17 137.1 mm to (74.9, 34.3)
- moved R13 135.1 mm to (64.8, 54.6), turned to 270 degrees
- moved C8 130.9 mm to (91.4, 72.4)
- moved R20 130.0 mm to (91.4, 55.9)
- moved Q15 123.6 mm to (47.0, 77.5)
- moved C9 120.5 mm to (91.4, 63.5)
- moved R12 118.7 mm to (61.0, 54.6), turned to 270 degrees
- moved D1 112.5 mm to (80.0, 72.4), flipped to the bottom
- moved R8 111.9 mm to (39.4, 36.8)
- moved Q12 108.0 mm to (43.2, 40.6)
- moved IC2 107.4 mm to (52.1, 55.9), turned to 90 degrees
- moved R19 104.5 mm to (85.1, 67.3), turned to 90 degrees
- moved R2 101.0 mm to (43.2, 43.2)
- moved Q2 99.4 mm to (30.5, 47.0), turned to 270 degrees
- moved Q8 94.7 mm to (43.2, 48.3)
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Routing:
- net +5V: track 0.00 -> 76.4 mm
- net N$3: track 0.00 -> 66.2 mm
- net N$5: track 0.00 -> 31.1 mm
- net N$4: track 0.00 -> 23.7 mm
- net N$2: track 0.00 -> 20.4 mm
- net N$7: track 0.00 -> 19.1 mm
- net N$12: track 0.00 -> 12.0 mm
- net N$8: track 0.00 -> 9.94 mm
- net N$13: track 0.00 -> 9.42 mm
- net GND: track 0.00 -> 8.15 mm
- net N$11: track 0.00 -> 7.62 mm
- net N$16: track 0.00 -> 5.08 mm
