File: LGM-01_pomocnicze/licznik.brd (EAGLE design)
At the start: 100 x 80 mm, 30 parts, among them IC1 7805L, J1 22-27-2041-04, Q3 BC557, T3 BC547, T4 BC547, T5 BC547

Commit message: Boards complete
Parts:
- moved PAD4 48.5 mm to (42.3, 2.54)
- moved PAD3 43.3 mm to (42.3, 6.35)
- moved R18 30.5 mm to (37.8, 38.1), turned to 90 degrees
- moved C2 30.5 mm to (28.9, 36.8)
- moved C4 30.5 mm to (17.5, 36.8)
- moved LED2 30.5 mm to (54.3, 36.8)
- moved LED3 30.5 mm to (54.3, 24.1), turned to 90 degrees
- moved T3 29.5 mm to (22.6, 8.89)
- moved C5 29.2 mm to (20.1, 45.7)
- moved J1 29.2 mm to (12.4, 45.7)
- moved IC1 29.2 mm to (22.6, 39.4)
- moved S1 29.2 mm to (39.1, 47.0)
- moved ZAS 29.2 mm to (51.8, 47.0)
- moved R10 27.0 mm to (32.8, 20.3)
- moved R21 27.0 mm to (37.8, 20.3)
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Routing:
- net N$17: track 96.1 -> 51.6 mm
- net VBAT: track 93.1 -> 76.6 mm
- net N$14: track 9.94 -> 23.0 mm
- net N$24: track 3.81 -> 16.5 mm
- net N$22: track 0.00 -> 8.15 mm
- net N$23: track 7.67 -> 14.2 mm
- net N$21: track 16.0 -> 21.7 mm
- net GND: track 230.6 -> 225.1 mm
- net +5V: track 93.2 -> 98.0 mm
- net WYJSCIE: track 28.0 -> 32.5 mm
- net N$18: track 16.9 -> 19.2 mm
- net KATODA: track 8.15 -> 9.94 mm
- net N$15: track 41.5 -> 39.7 mm
- net N$19: track 3.81 -> 2.54 mm
Other:
- board size 100 x 80 mm -> 60 x 54 mm
- board text added: "LGM-01-B"
- board text added: "MICHAL ZYCHLA 2024"

Commit message: Backup
Parts:
- moved R18 2.74 mm to (39.4, 40.4), turned to 180 degrees
- moved R5 1.42 mm to (9.26, 39.4)
Routing:
- net N$14: track 23.0 -> 13.0 mm
- net KATODA: track 9.94 -> 11.5 mm
- net N$17: track 51.6 -> 50.1 mm
- net WYJSCIE: track 32.5 -> 31.1 mm
Other:
- board text added: "Licznik G-M"
Changed lines of the file:
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@@
 <setting verticaltext="up"/>
 </settings>
-<grid distance="0.05" unitdist="inch" unit="inch" style="lines" multiple="1" display="no" altdistance="0.025" altunitdist="inch" altunit="inch"/>
+<grid distance="0.025" unitdist="inch" unit="inch" style="lines" multiple="1" display="no" altdistance="0.025" altunitdist="inch" altunit="inch"/>
 <layers>
 <layer number="1" name="Top" color="4" fill="1" visible="yes" active="yes"/>
@@
 <hole x="55" y="5" drill="3.2"/>
 <hole x="48" y="35" drill="3.2"/>
-<text x="45.72" y="29.21" size="1.778" layer="16" font="vector" ratio="15" rot="MR0">LGM-01-B</text>
-<text x="6.35" y="53.34" size="1.778" layer="16" font="vector" ratio="15" rot="MR180">MICHAL ZYCHLA 2024</text>
+<text x="59.055" y="52.07" size="1.778" layer="16" font="vector" ratio="15" rot="MR270">LGM-01-B</text>
+<text x="16.51" y="30.48" size="1.778" layer="16" font="vector" ratio="15" rot="MR180">MICHAL ZYCHLA 2024</text>
+<text x="57.15" y="9.525" size="1.778" layer="16" font="vector" ratio="15" rot="MR90">Licznik G-M</text>
 </plain>
 <attributes>
@@
 <element name="R15" library="resistor" package="0207/10" value="22k" x="12.43" y="7.62" rot="R90"/>
 <element name="R16" library="resistor" package="0207/10" value="470" x="17.51" y="20.32" rot="R270"/>
-<element name="R18" library="resistor" package="0207/10" value="1k" x="37.83" y="38.1" rot="R90"/>
-<element name="R5" library="resistor" package="0207/10" value="10k" x="9.89" y="40.64"/>
+<element name="R18" library="resistor" package="0207/10" value="1k" x="39.37" y="40.37" rot="R180"/>
+<element name="R5" library="resistor" package="0207/10" value="10k" x="9.255" y="39.37"/>
 <element name="R6" library="resistor" package="0207/10" value="100k" x="17.51" y="7.62" rot="R90"/>
 <element name="R7" library="resistor" package="0207/10" value="100k" x="22.59" y="20.32" rot="R90"/>
@@
 <wire x1="28.94" y1="34.29" x2="23.86" y2="34.29" width="0.6096" layer="16"/>
 <wire x1="23.86" y1="34.29" x2="22.59" y2="35.56" width="0.6096" layer="16"/>
-<wire x1="6.08" y1="50.8" x2="16.24" y2="50.8" width="0.6096" layer="16"/>
 <wire x1="16.24" y1="50.8" x2="22.59" y2="50.8" width="0.6096" layer="16"/>
 <wire x1="22.59" y1="50.8" x2="28.94" y2="50.8" width="0.6096" layer="16"/>
@@
 <wire x1="44.54" y1="2.54" x2="50.165" y2="8.165" width="0.6096" layer="16"/>
 <wire x1="50.165" y1="11.0038" x2="50.165" y2="8.165" width="0.6096" layer="16"/>
-<wire x1="17.51" y1="2.54" x2="19.05" y2="2.54" width="0.6096" layer="16"/>
-<wire x1="19.05" y1="2.54" x2="19.685" y2="3.175" width="0.6096" layer="16"/>
-<wire x1="19.685" y1="3.175" x2="21.59" y2="5.08" width="0.6096" layer="16"/>
-<wire x1="21.59" y1="5.08" x2="21.59" y2="6.62" width="0.6096" layer="16"/>
-<wire x1="21.59" y1="6.62" x2="22.59" y2="7.62" width="0.6096" layer="16"/>
-<wire x1="21.59" y1="5.08" x2="25.4" y2="5.08" width="0.6096" layer="16"/>
-<wire x1="25.4" y1="5.08" x2="27.94" y2="2.54" width="0.6096" layer="16"/>
-<wire x1="27.94" y1="2.54" x2="37.83" y2="2.54" width="0.6096" layer="16"/>
-<wire x1="25.4" y1="5.08" x2="25.4" y2="5.35" width="0.6096" layer="16"/>
-<wire x1="25.4" y1="5.35" x2="27.67" y2="7.62" width="0.6096" layer="16"/>
 <wire x1="25.892" y1="45.72" x2="24.13" y2="45.72" width="0.6096" layer="16"/>
 <wire x1="24.13" y1="45.72" x2="22.59" y2="44.18" width="0.6096" layer="16"/>
 <wire x1="22.59" y1="41.275" x2="22.59" y2="44.18" width="0.6096" layer="16"/>
 <wire x1="2.27" y1="12.97" x2="10.16" y2="5.08" width="0.6096" layer="16"/>
-<wire x1="10.16" y1="5.08" x2="17.78" y2="5.08" width="0.6096" layer="16"/>
-<wire x1="17.78" y1="5.08" x2="19.685" y2="3.175" width="0.6096" layer="16"/>
+<wire x1="6.08" y1="50.8" x2="16.24" y2="50.8" width="0.6096" layer="16"/>
+<wire x1="10.16" y1="5.08" x2="10.16" y2="3.175" width="0.6096" layer="16"/>
+<wire x1="10.16" y1="3.175" x2="10.795" y2="2.54" width="0.6096" layer="16"/>
+<wire x1="10.795" y1="2.54" x2="12.43" y2="2.54" width="0.6096" layer="16"/>
 <wire x1="12.43" y1="2.54" x2="17.51" y2="2.54" width="0.6096" layer="16"/>
+<wire x1="10.16" y1="5.08" x2="12.7" y2="7.62" width="0.6096" layer="16"/>
+<wire x1="22.59" y1="7.62" x2="12.7" y2="7.62" width="0.6096" layer="16"/>
+<wire x1="22.59" y1="7.62" x2="22.86" y2="7.62" width="0.6096" layer="16"/>
+<wire x1="22.86" y1="7.62" x2="24.765" y2="5.715" width="0.6096" layer="16"/>
+<wire x1="24.765" y1="5.715" x2="27.94" y2="2.54" width="0.6096" layer="16"/>
+<wire x1="27.94" y1="2.54" x2="37.83" y2="2.54" width="0.6096" layer="16"/>
+<wire x1="27.67" y1="7.62" x2="26.67" y2="7.62" width="0.6096" layer="16"/>
+<wire x1="26.67" y1="7.62" x2="24.765" y2="5.715" width="0.6096" layer="16"/>
 </signal>
 <signal name="+5V">
@@
 <wire x1="28.94" y1="45.212" x2="29.448" y2="45.72" width="0.6096" layer="16"/>
 <wire x1="29.448" y1="45.72" x2="32.75" y2="45.72" width="0.6096" layer="16"/>
-<wire x1="32.75" y1="45.72" x2="35.29" y2="43.18" width="0.6096" layer="16"/>
-<wire x1="35.29" y1="43.18" x2="37.83" y2="43.18" width="0.6096" layer="16"/>
 <wire x1="35.29" y1="46.99" x2="34.02" y2="46.99" width="0.6096" layer="16"/>
 <wire x1="34.02" y1="46.99" x2="32.75" y2="45.72" width="0.6096" layer="16"/>
@@
 <wire x1="11.16" y1="31.75" x2="8.62" y2="34.29" width="0.6096" layer="16"/>
 <wire x1="11.16" y1="31.75" x2="8.62" y2="29.21" width="0.6096" layer="16"/>
+<wire x1="32.75" y1="45.72" x2="33.02" y2="45.72" width="0.6096" layer="16"/>
+<wire x1="33.02" y1="45.72" x2="34.29" y2="44.45" width="0.6096" layer="16"/>
+<wire x1="34.29" y1="44.45" x2="34.29" y2="40.37" width="0.6096" layer="16"/>
 </signal>
 <signal name="N$17">
@@
 <contactref element="R6" pad="2"/>
 <contactref element="T3" pad="2"/>
-<wire x1="4.81" y1="40.64" x2="4.175" y2="40.005" width="0.6096" layer="16"/>
-<wire x1="4.175" y1="40.005" x2="4.175" y2="14.605" width="0.6096" layer="16"/>
+<wire x1="4.175" y1="39.37" x2="4.175" y2="40.005" width="0" layer="19" extent="1-16"/>
+<wire x1="4.175" y1="39.37" x2="4.175" y2="14.605" width="0.6096" layer="16"/>
 <wire x1="4.175" y1="14.605" x2="9.255" y2="9.525" width="0.6096" layer="16"/>
 <wire x1="9.255" y1="9.525" x2="11.795" y2="9.525" width="0.6096" layer="16"/>
@@
 <contactref element="J1" pad="4"/>
 <wire x1="16.24" y1="45.72" x2="16.24" y2="41.91" width="0.6096" layer="16"/>
-<wire x1="16.24" y1="41.91" x2="14.97" y2="40.64" width="0.6096" layer="16"/>
 <wire x1="20.05" y1="43.18" x2="17.51" y2="43.18" width="0.6096" layer="16"/>
 <wire x1="17.51" y1="43.18" x2="16.24" y2="41.91" width="0.6096" layer="16"/>
+<wire x1="14.335" y1="39.37" x2="14.335" y2="40.005" width="0.6096" layer="16"/>
+<wire x1="14.335" y1="40.005" x2="16.24" y2="41.91" width="0.6096" layer="16"/>
 </signal>
 <signal name="N$15">
@@
 <contactref element="LED2" pad="A"/>
 <contactref element="R18" pad="1"/>
-<wire x1="54.34" y1="35.56" x2="53.07" y2="35.56" width="0.6096" layer="16"/>
-<wire x1="53.07" y1="35.56" x2="49.26" y2="39.37" width="0.6096" layer="16"/>
-<wire x1="49.26" y1="39.37" x2="44.18" y2="39.37" width="0.6096" layer="16"/>
-<wire x1="44.18" y1="39.37" x2="42.91" y2="38.1" width="0.6096" layer="16"/>
-<wire x1="42.91" y1="38.1" x2="42.91" y2="34.29" width="0.6096" layer="16"/>
-<wire x1="42.91" y1="34.29" x2="41.64" y2="33.02" width="0.6096" layer="16"/>
-<wire x1="41.64" y1="33.02" x2="37.83" y2="33.02" width="0.6096" layer="16"/>
+<wire x1="44.45" y1="40.37" x2="49.165" y2="40.37" width="0.6096" layer="16"/>
+<wire x1="49.165" y1="40.37" x2="51.435" y2="38.1" width="0.6096" layer="16"/>
+<wire x1="51.435" y1="38.1" x2="51.435" y2="36.195" width="0.6096" layer="16"/>
+<wire x1="51.435" y1="36.195" x2="52.07" y2="35.56" width="0.6096" layer="16"/>
+<wire x1="52.07" y1="35.56" x2="54.34" y2="35.56" width="0.6096" layer="16"/>
 </signal>
 <signal name="N$19">
@@
 <wire x1="42.275" y1="6.715" x2="46.99" y2="11.43" width="0.6096" layer="16"/>
 <wire x1="46.99" y1="11.43" x2="46.99" y2="14.9662" width="0.6096" layer="16"/>
-<wire x1="46.99" y1="14.9662" x2="44.45" y2="17.5062" width="0.6096" layer="16"/>
-<wire x1="44.45" y1="17.5062" x2="50.165" y2="17.5062" width="0.6096" layer="16"/>
+<wire x1="46.99" y1="14.9662" x2="46.8531" y2="15.1031" width="0.6096" layer="16"/>
+<wire x1="46.8531" y1="15.1031" x2="44.45" y2="17.5062" width="0.6096" layer="16"/>
+<wire x1="50.165" y1="17.5062" x2="49.2562" y2="17.5062" width="0.6096" layer="16"/>
+<wire x1="49.2562" y1="17.5062" x2="46.8531" y2="15.1031" width="0.6096" layer="16"/>
 </signal>
 <signal name="N$21">
